Commit message: iliad robot

File: vito_description/model/torso.urdf.xacro (robot description, xacro)
@@ -28,5 +28,5 @@
       </geometry>
       <material name="Vito/Silver"/>
-    </visual>
+    </visual>z
     <collision>
       <geometry>
@@ -38,4 +38,28 @@
     <!-- <static>true</static> -->
   </gazebo>
+<joint name="${parent}_${name}_base_joint_b" type="fixed">
+    <origin xyz="-0.09 0.0 0.49" rpy="${pi / 2} 0 0"/>
+    <parent link="${name}_link"/>
+    <child link="${name}_link_b"/>
+  </joint>
+  <link name="${name}_link_b">
+    <inertial>
+      <xacro:insert_block name="torso_inertia"/>
+    </inertial>
+    <visual>
+      <geometry>
+        <mesh filename="package://vito_description/meshes/torso_b.stl"/>
+      </geometry>
+      <material name="Vito/Silver"/>
+    </visual>z
+    <collision>
+      <geometry>
+        <mesh filename="package://vito_description/meshes/torso_b.stl"/>
+      </geometry>
+    </collision>
+  </link>
+  <gazebo reference="${name}_link_b">
+    <!-- <static>true</static> -->
+  </gazebo>
 </xacro:macro>
 </robot>

File: vito_description/robot/vito.urdf.xacro (robot description, xacro)
@@ -22,5 +22,5 @@
                     height="0.910"
                     plate_thickness="0.05">
-    <origin xyz="-0.495 0.55 0" rpy="0 0 0"/>
+    <origin xyz="0.0 0.55 0" rpy="0 0 0"/>
   </xacro:model_table>
   <!-- WORKBENCH -->
